File: KiCad/LoKiPAD.kicad_pcb (KiCad board)
At the start: 2 copper layers, 60 x 100 mm, 64 parts, among them J1 AudioJack4, J2 Conn_01x07_Female, J3 AudioJack4, SW1 SW_Push, SW10 SW_Push, SW11 SW_Push, SW12 SW_Push, SW13 Rotary_Encoder_Switch, SW2 SW_Push, SW3 SW_Push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

Commit message: more parts moved to back, kicad7
Parts:
- added J4: Conn_01x04_Socket, Connector_JST:JST_SH_BM04B-SRSS-TB_1x04-1MP_P1.00mm_Vertical, B.Cu at (48.9, 2.57)
- added R10: 4.7k, Resistor_SMD:R_0603_1608Metric_Pad0.98x0.95mm_HandSolder, B.Cu at (54.4, 5.62)
- added R9: 4.7k, Resistor_SMD:R_0603_1608Metric_Pad0.98x0.95mm_HandSolder, B.Cu at (54.4, 3.84)
- added SW14: SW_Push, Button_Switch_SMD:SW_Push_1P1T_NO_CK_KMR2, F.Cu at (49.7, 3.62)
- added U3: MCP73831-2-OT, Package_TO_SOT_SMD:SOT-23-5, B.Cu at (50.3, 93.1)
- C13, C14, C15, D14, J1, J3, R2, R3, R4, R5, R6, U2: moved to B.Cu
- moved kibuzzard-63E7EF8E 9.45 mm to (3.13, 20.4), turned to -90 degrees
- moved C13 7.93 mm to (32.4, 28.4), turned to -90 degrees
- moved R2 7.93 mm to (15.6, 28.4), turned to 90 degrees
- moved kibuzzard-63D67711 7.48 mm to (1.36, 21.9), turned to -90 degrees
- moved kibuzzard-63D67702 7.04 mm to (1.36, 8.41), turned to -90 degrees
- moved R3 2.51 mm to (32.4, 23.2), turned to -90 degrees
- moved D14 1.15 mm to (15.6, 23.9), turned to 90 degrees
- moved U2 0.99 mm to (24.1, 24.9)
- moved C14 0.15 mm to (19.9, 9.94), turned to 90 degrees
- moved C15 0.15 mm to (15.9, 9.94), turned to -90 degrees
- moved R4 0.15 mm to (21.9, 9.94), turned to -90 degrees
- moved R5 0.15 mm to (13.9, 9.94), turned to -90 degrees
- moved R6 0.15 mm to (17.9, 9.94), turned to 90 degrees
Connections:
- U1 pad 17: LED -> real_SCL
- U1 pad 21: unconnected-(U1-Pad21) -> real_SDA
- U1 pad 30: unconnected-(U1-Pad30) -> run
Routing:
- net run: track 0.00 -> 105.3 mm, vias 0 -> 3
- net real_SCL: track 0.00 -> 86.7 mm, vias 0 -> 2
- net real_SDA: track 0.00 -> 63.0 mm
- net SCL: track 57.3 -> 67.9 mm, vias 1 -> 2
- net SDA: track 71.8 -> 80.0 mm, vias 1 -> 2
- net VCC: track 380.9 -> 387.0 mm, vias 4 -> 6
- net DS_DATA: track 83.0 -> 86.3 mm
- net DS_CS: track 72.1 -> 74.4 mm
- net DS_DC: track 54.5 -> 52.8 mm
- net Net-(D14-A): track 15.1 -> 13.5 mm
- net DS_CLK: track 85.7 -> 87.1 mm
- net Net-(J1-PadR1): track 12.5 -> 11.2 mm
- net DS_RES: track 50.3 -> 49.3 mm
- net GND: vias 56 -> 60
